File: Board/ESC/Brushless_ESC.kicad_pcb (KiCad board)
At the start: 2 copper layers, 63 x 36 mm, 77 parts, among them IC1 ATMEGA88PA-A, P1 Battery+, P10 MISO, P11 Reset, P12 SCK, P13 Gnd, P2 Battery-, P3 Coil_A, P4 Sup, P5 Coil_B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

Commit message: Layout Fehler (LED an ADC7) behoben
Parts:
- turned R1 to 0 degrees
Connections:
- C4 pad 1: +5V -> Net-(C4-Pad1)
- IC1 pad 20: +5V -> Net-(C4-Pad1)
- IC1 pad 22: Net-(IC1-Pad22) -> /Controller/V_Bat
- IC1 pad 23: /Controller/V_Bat -> Net-(IC1-Pad23)
- R1 pad 1: Net-(IC1-Pad22) -> Net-(D1-Pad2)
- R1 pad 2: Net-(D1-Pad2) -> Net-(IC1-Pad23)
Routing:
- net Net-(IC1-Pad23): track 0.00 -> 17.2 mm
- net Net-(IC1-Pad22): track 15.4 -> 0.00 mm
- net +5V: track 69.9 -> 63.0 mm
- net Net-(C4-Pad1): track 0.00 -> 3.39 mm
- net /Controller/V_Bat: track 34.4 -> 31.5 mm
Changed lines of the file:
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@@
 (kicad_pcb (version 4) (host pcbnew 4.0.0-rc1-stable)
   (general
-    (links 138)
+    (links 137)
     (no_connects 0)
     (area 104.839501 51.569515 179.406001 97.241)
     (thickness 1.6)
     (drawings 15)
-    (tracks 473)
+    (tracks 472)
     (zones 0)
     (modules 77)
-    (nets 53)
+    (nets 54)
   )
   (page A4)
@@
   (net 50 FET_Drain)
   (net 51 "Net-(IC1-Pad18)")
-  (net 52 "Net-(IC1-Pad22)")
+  (net 52 "Net-(C4-Pad1)")
+  (net 53 "Net-(IC1-Pad23)")
   (net_class Default "Dies ist die voreingestellte Netzklasse."
     (clearance 0.2)
@@
     (add_net "Net-(C12-Pad1)")
     (add_net "Net-(C16-Pad1)")
+    (add_net "Net-(C4-Pad1)")
     (add_net "Net-(C6-Pad1)")
     (add_net "Net-(C7-Pad2)")
@@
     (add_net "Net-(IC1-Pad17)")
     (add_net "Net-(IC1-Pad18)")
-    (add_net "Net-(IC1-Pad22)")
+    (add_net "Net-(IC1-Pad23)")
     (add_net "Net-(IC1-Pad29)")
     (add_net "Net-(Q1-Pad1)")
@@
     (pad 19 smd rect (at 4.25 1.2 270) (size 1.6 0.55) (layers F.Cu F.Paste F.Mask))
     (pad 20 smd rect (at 4.25 0.4 270) (size 1.6 0.55) (layers F.Cu F.Paste F.Mask)
-      (net 1 +5V))
+      (net 52 "Net-(C4-Pad1)"))
     (pad 21 smd rect (at 4.25 -0.4 270) (size 1.6 0.55) (layers F.Cu F.Paste F.Mask)
       (net 2 GND))
     (pad 22 smd rect (at 4.25 -1.2 270) (size 1.6 0.55) (layers F.Cu F.Paste F.Mask)
-      (net 52 "Net-(IC1-Pad22)"))
+      (net 22 /Controller/V_Bat))
     (pad 23 smd rect (at 4.25 -2 270) (size 1.6 0.55) (layers F.Cu F.Paste F.Mask)
-      (net 22 /Controller/V_Bat))
+      (net 53 "Net-(IC1-Pad23)"))
     (pad 24 smd rect (at 4.25 -2.8 270) (size 1.6 0.55) (layers F.Cu F.Paste F.Mask)
       (net 45 /Controller/BatCurrent+))
@@
   )
   (module Resistors_SMD:R_0805_HandSoldering (layer F.Cu)
-    (at 128.0795 89.789 180)
+    (at 128.0795 89.789)
     (descr "Resistor SMD 0805, hand soldering")
     (tags "resistor 0805")
     (attr smd)
-    (fp_text reference R1 (at 0 -2.032 180) (layer F.SilkS)
-      (effects (font (size 1 1) (thickness 0.15)))
-    )
-    (fp_text value 220R (at 0 2.1 180) (layer F.Fab)
+    (fp_text reference R1 (at 0 -2.032) (layer F.SilkS)
+      (effects (font (size 1 1) (thickness 0.15)))
+    )
+    (fp_text value 220R (at 0 2.1) (layer F.Fab)
       (effects (font (size 1 1) (thickness 0.15)))
     )
@@
     (fp_line (start 0.6 0.875) (end -0.6 0.875) (layer F.SilkS) (width 0.15))
     (fp_line (start -0.6 -0.875) (end 0.6 -0.875) (layer F.SilkS) (width 0.15))
-    (pad 1 smd rect (at -1.35 0 180) (size 1.5 1.3) (layers F.Cu F.Paste F.Mask)
-      (net 52 "Net-(IC1-Pad22)"))
-    (pad 2 smd rect (at 1.35 0 180) (size 1.5 1.3) (layers F.Cu F.Paste F.Mask)
+    (pad 1 smd rect (at -1.35 0) (size 1.5 1.3) (layers F.Cu F.Paste F.Mask)
       (net 15 "Net-(D1-Pad2)"))
+    (pad 2 smd rect (at 1.35 0) (size 1.5 1.3) (layers F.Cu F.Paste F.Mask)
+      (net 53 "Net-(IC1-Pad23)"))
     (model Resistors_SMD.3dshapes/R_0805_HandSoldering.wrl
       (at (xyz 0 0 0))
@@
     (fp_line (start 0.35 0.6) (end -0.35 0.6) (layer F.SilkS) (width 0.15))
     (pad 1 smd rect (at -0.95 0 270) (size 1.2 0.75) (layers F.Cu F.Paste F.Mask)
-      (net 1 +5V))
+      (net 52 "Net-(C4-Pad1)"))
     (pad 2 smd rect (at 0.95 0 270) (size 1.2 0.75) (layers F.Cu F.Paste F.Mask)
       (net 2 GND))
@@
   (via (at 128.0795 86.106) (size 1) (drill 0.8) (layers F.Cu B.Cu) (net 1))
   (segment (start 129.2835 87.31) (end 128.0795 86.106) (width 0.25) (layer F.Cu) (net 1))
-  (segment (start 137.0965 85.664) (end 137.0965 86.106) (width 0.25) (layer F.Cu) (net 1) (status 30))
-  (segment (start 137.0965 86.106) (end 136.2075 86.995) (width 0.25) (layer F.Cu) (net 1) (status 10))
-  (segment (start 136.2075 86.995) (end 133.9215 86.995) (width 0.25) (layer F.Cu) (net 1) (status 20))
   (segment (start 123.7615 70.612) (end 121.9835 70.612) (width 0.25) (layer F.Cu) (net 1))
   (segment (start 119.1895 70.612) (end 121.539 70.612) (width 0.25) (layer F.Cu) (net 1) (status 10))
@@
   (segment (start 136.2775 74.744) (end 136.2775 71.492) (width 0.25) (layer F.Cu) (net 1) (status 30))
   (segment (start 136.2775 71.492) (end 136.4615 71.308) (width 0.25) (layer F.Cu) (net 1) (status 30))
-  (segment (start 137.0965 85.664) (end 137.0965 83.263) (width 0.25) (layer F.Cu) (net 1) (status 30))
-  (segment (start 137.0965 83.263) (end 137.0775 83.244) (width 0.25) (layer F.Cu) (net 1) (status 30))
   (segment (start 131.6355 87.31) (end 133.6065 87.31) (width 0.25) (layer F.Cu) (net 1) (status 30))
-  (segment (start 136.9695 83.352) (end 137.0775 83.244) (width 0.25) (layer F.Cu) (net 1) (status 30))
-  (segment (start 136.9695 83.352) (end 137.0775 83.244) (width 0.25) (layer F.Cu) (net 1) (status 30))
-  (segment (start 136.9695 83.352) (end 137.0775 83.244) (width 0.25) (layer F.Cu) (net 1) (status 30))
-  (segment (start 137.11936 83.28586) (end 137.0775 83.244) (width 0.25) (layer F.Cu) (net 1) (status 30))
   (segment (start 128.3335 68.6) (end 128.3335 67.691) (width 0.25) (layer F.Cu) (net 2))
   (via (at 129.3495 66.675) (size 1) (drill 0.8) (layers F.Cu B.Cu) (net 2))
@@
   (segment (start 170.6372 89.93124) (end 173.53026 89.93124) (width 0.25) (layer B.Cu) (net 14) (status 10))
   (segment (start 173.53026 89.93124) (end 175.8315 87.63) (width 0.25) (layer B.Cu) (net 14) (status 20))
-  (segment (start 120.74652 89.789) (end 123.3805 89.789) (width 0.25) (layer F.Cu) (net 15))
-  (segment (start 123.3805 89.789) (end 126.7295 89.789) (width 0.25) (layer F.Cu) (net 15) (status 10))
+  (segment (start 120.74652 89.789) (end 126.7295 89.789) (width 0.25) (layer F.Cu) (net 15) (status C00000))
   (segment (start 119.1895 79.756) (end 122.475 79.756) (width 0.25) (layer F.Cu) (net 16) (status 30))
   (segment (start 119.1895 77.47) (end 122.475 77.47) (width 0.25) (layer F.Cu) (net 17) (status 30))
@@
   (segment (start 133.905 77.216) (end 133.905 79.502) (width 0.25) (layer B.Cu) (net 21) (status 30))
   (segment (start 133.905 81.788) (end 133.905 79.502) (width 0.25) (layer B.Cu) (net 21) (status 30))
-  (segment (start 121.7495 80.01) (end 121.7495 83.078) (width 0.25) (layer B.Cu) (net 22))
-  (segment (start 139.4775 87.852) (end 140.2715 88.646) (width 0.25) (layer F.Cu) (net 22))
-  (segment (start 139.4775 87.852) (end 139.4775 83.244) (width 0.25) (layer F.Cu) (net 22) (status 10))
-  (via (at 140.2715 88.646) (size 1) (drill 0.8) (layers F.Cu B.Cu) (net 22))
+  (segment (start 138.6775 83.244) (end 138.6775 86.925) (width 0.25) (layer F.Cu) (net 22) (status 400000))
+  (segment (start 121.7495 83.078) (end 124.2495 85.578) (width 0.25) (layer B.Cu) (net 22))
   (segment (start 124.2495 85.578) (end 126.3015 87.63) (width 0.25) (layer B.Cu) (net 22))
-  (segment (start 126.3015 87.63) (end 139.2555 87.63) (width 0.25) (layer B.Cu) (net 22))
-  (segment (start 139.2555 87.63) (end 140.2715 88.646) (width 0.25) (layer B.Cu) (net 22))
-  (segment (start 121.7495 83.078) (end 124.2495 85.578) (width 0.25) (layer B.Cu) (net 22))
+  (segment (start 121.7495 83.078) (end 121.7495 80.01) (width 0.25) (layer B.Cu) (net 22))
+  (segment (start 138.8745 87.63) (end 126.3015 87.63) (width 0.25) (layer B.Cu) (net 22))
+  (segment (start 139.1285 87.376) (end 138.8745 87.63) (width 0.25) (layer B.Cu) (net 22))
+  (via (at 139.1285 87.376) (size 1) (drill 0.8) (layers F.Cu B.Cu) (net 22))
+  (segment (start 138.6775 86.925) (end 139.1285 87.376) (width 0.25) (layer F.Cu) (net 22))
   (segment (start 121.7295 77.55) (end 121.7295 79.99) (width 0.25) (layer B.Cu) (net 22))
   (segment (start 121.7295 79.99) (end 121.7495 80.01) (width 0.25) (layer B.Cu) (net 22))
@@
   (segment (start 135.1915 85.217) (end 135.4775 84.931) (width 0.25) (layer F.Cu) (net 51))
   (segment (start 135.4455 83.276) (end 135.4775 83.244) (width 0.25) (layer F.Cu) (net 51) (status 30))
-  (segment (start 129.4295 89.789) (end 137.9855 89.789) (width 0.25) (layer F.Cu) (net 52) (status 10))
-  (segment (start 138.6775 89.097) (end 138.6775 83.244) (width 0.25) (layer F.Cu) (net 52) (status 20))
-  (segment (start 137.9855 89.789) (end 138.6775 89.097) (width 0.25) (layer F.Cu) (net 52))
+  (segment (start 137.0965 85.664) (end 137.0965 86.106) (width 0.25) (layer F.Cu) (net 52) (status 30))
+  (segment (start 137.0965 85.664) (end 137.0965 83.263) (width 0.25) (layer F.Cu) (net 52) (status 30))
+  (segment (start 137.0965 83.263) (end 137.0775 83.244) (width 0.25) (layer F.Cu) (net 52) (status 30))
+  (segment (start 136.9695 83.352) (end 137.0775 83.244) (width 0.25) (layer F.Cu) (net 52) (status 30))
+  (segment (start 136.9695 83.352) (end 137.0775 83.244) (width 0.25) (layer F.Cu) (net 52) (status 30))
+  (segment (start 136.9695 83.352) (end 137.0775 83.244) (width 0.25) (layer F.Cu) (net 52) (status 30))
+  (segment (start 137.11936 83.28586) (end 137.0775 83.244) (width 0.25) (layer F.Cu) (net 52) (status 30))
+  (segment (start 129.4295 89.789) (end 139.0015 89.789) (width 0.25) (layer F.Cu) (net 53) (status 400000))
+  (segment (start 139.4775 85.693) (end 139.4775 83.244) (width 0.25) (layer F.Cu) (net 53) (status 800000))
+  (segment (start 140.5255 86.741) (end 139.4775 85.693) (width 0.25) (layer F.Cu) (net 53))
+  (segment (start 140.5255 88.265) (end 140.5255 86.741) (width 0.25) (layer F.Cu) (net 53))
+  (segment (start 139.0015 89.789) (end 140.5255 88.265) (width 0.25) (layer F.Cu) (net 53))
   (zone (net 2) (net_name GND) (layer B.Cu) (hatch edge 0.508)
     (connect_pads yes (clearance 0.254))

Commit message: Minor Layout changes
Parts:
- moved R23 2.42 mm to (126.4, 76.3)
- moved C17 2.16 mm to (125.2, 79.9)
- moved R22 2.16 mm to (123.9, 76.3)
Routing:
- net +5V: track 63.0 -> 65.2 mm
- net /Controller/V_Bat: track 31.5 -> 30.4 mm
Other:
- board text added: "ESC v1.5"
- board text removed: "ESC v1.0"
