File: Board/ESC/Brushless_ESC.kicad_pcb (KiCad board)
At the start: 2 copper layers, 63 x 36 mm, 76 parts, among them IC1 ATMEGA88PA-A, P1 Battery+, P2 Battery-, P3 Coil_A, P4 PPM, P5 Coil_B, P6 Coil_C, P7 I2C, P8 ISP, Q1 IRL7843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

Commit message: Layoutänderung
Parts:
- moved D2 4.71 mm to (124.9, 77.0), turned to 180 degrees
- moved C2 2.90 mm to (132.4, 85.7), turned to 90 degrees
- moved C3 1.27 mm to (138.5, 71.2)
- moved C6 1.09 mm to (131.8, 67.7)
- moved C7 0.76 mm to (127.3, 69.8)
- moved Y1 0.76 mm to (131.6, 70.7)
- moved C21 0.51 mm to (126.4, 70.7)
- moved L1 0.28 mm to (126.6, 85.9)
- moved C4 0.25 mm to (138.9, 87.2)
Connections:
- U1 pad 10: (no net) -> GND
- U1 pad 11: (no net) -> GND
- U1 pad 12: (no net) -> GND
- U1 pad 4: (no net) -> GND
- U1 pad 5: (no net) -> GND
Routing:
- net GND: track 27.4 -> 44.5 mm
- net +5V: track 69.7 -> 75.9 mm
- net /Controller/PPM: track 16.5 -> 14.0 mm
- net /Controller/SCL: track 33.5 -> 31.1 mm
- net /Controller/V_Bat: track 55.4 -> 57.2 mm
- net /Controller/SDA: track 33.7 -> 32.5 mm
- net Net-(C7-Pad2): track 9.74 -> 10.8 mm
- net Net-(C2-Pad1): track 10.3 -> 11.3 mm
- net /Controller/T_Sense: track 56.8 -> 56.2 mm
- net /Controller//SD_A: track 30.0 -> 29.5 mm

Commit message: Final Layout
Parts:
- added G***: LOGO, Loewe:Loewe_Klein, F.Cu at (145.7, 81.8)
- D4, D5, D6: footprint w_smd_diode:sod123 -> Diodes_SMD:SOD-123
- Q1, Q2, Q3, Q4, Q5, Q6: footprint w_smd_trans:d-pak -> TO_SOT_Packages_SMD:TO-252-2Lead
- U2, U3, U4: footprint w_smd_dil:so-8 -> Housings_SOIC:SOIC-8_3.9x4.9mm_Pitch1.27mm
- moved Q2 3.18 mm to (162.9, 64.3)
- moved Q4 3.18 mm to (162.9, 75.7)
- moved Q6 3.18 mm to (162.9, 87.5)
- moved Q1 3.05 mm to (170.1, 64.3)
- moved Q3 3.05 mm to (170.1, 75.6)
- moved Q5 2.92 mm to (170.0, 87.5)
- moved C12 0.65 mm to (153.0, 79.8), turned to 0 degrees
- moved C11 0.54 mm to (152.9, 69.8), turned to 0 degrees
- moved U2 0.19 mm to (150.1, 63.8), turned to 0 degrees
- moved U3 0.10 mm to (150.1, 73.7), turned to 0 degrees
- moved U4 0.10 mm to (150.1, 83.8), turned to 0 degrees
Routing:
- net (no net): track 0.00 -> 16.0 mm
- net GND: track 44.5 -> 57.7 mm, vias 6 -> 9
- net /Power/Coil_B: track 39.3 -> 35.6 mm, vias 2 -> 3
- net /Power/Coil_A: track 36.9 -> 35.5 mm, vias 2 -> 3
- net Net-(R5-Pad2): track 25.1 -> 24.1 mm
- net Net-(R7-Pad2): track 16.9 -> 16.0 mm
- net /Controller/SDA: track 32.5 -> 31.6 mm
- net Net-(C12-Pad1): track 5.99 -> 5.30 mm
